Commit message: simulation fixed small issues and trying stuff

File: isaac_ros-dev/src/autonav_sim/description/custom_robot/camera.xacro (robot description, xacro)
@@ -13,9 +13,14 @@
             <material name="red"/>
         </visual>
+        <inertial>
+            <mass value="0.1"/>
+            <origin xyz="0 0 0" rpy="0 0 0"/>
+            <inertia ixx="0.0001" ixy="0.0" ixz="0.0" iyy="0.00001" iyz="0.0" izz="0.00001"/>
+        </inertial>
     </link>
     <joint name="camera_optical_joint" type="fixed">
         <parent link="camera_link"/>
         <child link="camera_link_optical"/>
-        <origin xyz="0 0 0" rpy="${-pi/2} 0 ${-pi/2}"/>
+        <origin xyz="0 0 0" rpy="${-pi/2} ${-pi/4} ${-pi/2}"/>
     </joint>
     <link name="camera_link_optical"></link>

File: isaac_ros-dev/src/autonav_sim/description/custom_robot/robot_core.xacro (robot description, xacro)
@@ -13,4 +13,7 @@
     <material name="black">
         <color rgba="0 0 0 1"/>
+    </material>
+    <material name="red">
+        <color rgba="1 0 0 1"/>
     </material>
     <!--START OF BASE LINK-->
@@ -46,4 +49,9 @@
             <origin xyz="0 0 0" rpy="0 0 0"/>
         </xacro:inertial_box>
+        <inertial>
+            <mass value="5.0"/>
+            <origin xyz="0 0 0" rpy="0 0 0"/>
+            <inertia ixx="0.1" ixy="0.0" ixz="0.0" iyy="0.1" iyz="0.0" izz="0.1"/>
+        </inertial>
     </link>
     <gazebo reference="chassis">
@@ -52,5 +60,5 @@
     <!--END OF CHASSIS MODEL-->
     <!--END OF CHASSIS LINK-->
-    <!--START OF LEFT WHEEL LINK-->
+    <!--START OF LEFT Wros2 lauros2 launch autonav_sim launch_sim.launch.py world:=./src/autonav_sim/worlds/autonav_igvc_course.worldnch autonav_sim launch_sim.launch.py world:=./src/autonav_sim/worlds/autonav_igvc_course.worldHEEL LINK-->
     <joint name="left_wheel_joint" type="continuous">
         <parent link="base_link"/>
