Commit message: sim stuff

File: isaac_ros-dev/src/sim/description/custom_robot/imu.xacro (robot description, xacro)
@@ -1,27 +1,34 @@
 <?xml version="1.0"?>
-<robot xmlns:xacro="http://www.ros.org/wiki/xacro" >
-    <joint name='imu_joint' type='fixed'>
-        <parent>base_link</parent>
-        <child>imu_link</child>
-        <pose relative_to="base_link">0.0 0.0 0.01 0 0 0</pose>
-    </joint>
+<robot xmlns:xacro="http://www.ros.org/wiki/xacro">
+    <xacro:include filename="inertial_macros.xacro"/>
     <link name='imu_link'>
-        <pose relative_to="imu_joint"/>
         <visual name="imu_link_visual">
             <geometry>
-                <box><size>
-                    0.1 0.1 0.1
-                </size></box>
+                <box size="0.1 0.1 0.1"/>
             </geometry>
         </visual>
         <collision name="imu_link_collision">
             <geometry>
-                <box><size>
-                    0.1 0.1 0.1
-                </size></box>
+                <box size="0.1 0.1 0.1"/>
             </geometry>
         </collision>
-        <xacro:box_inertia m="0.1" w="0.1" d="0.1" h="0.1"/>
+        <xacro:inertial_box mass="0.5" x="0.8636" y="0.4572" z="0.41021">
+            <origin xyz="0 0 0" rpy="0 0 0"/>
+        </xacro:inertial_box>
+    </link>
+    <joint name='imu_joint' type='fixed'>
+        <parent link="base_link"/>
+        <child link="imu_link"/>
+        <pose relative_to="base_link">0.0 0.0 0.01 0 0 0</pose>
+    </joint>
+    <gazebo reference="imu_link">
         <sensor name="imu_sensor" type="imu">
+            <plugin filename="libgazebo_ros_imu_sensor.so" name="imu_plugin">
+                <ros>
+                    <namespace>/autonav</namespace>
+                    <remapping>~/out:=/imu</remapping>
+                </ros>
+                <initial_orientation_as_reference>false</initial_orientation_as_reference>
+            </plugin>
             <always_on>true</always_on>
             <update_rate>100</update_rate>
@@ -84,26 +91,4 @@
             </imu>
         </sensor>
-    </link>
-    <plugin filename="gz-sim-diff-drive-system" name="gz::sim::systems::DiffDrive">
-        <!-- wheels -->
-        <left_joint>drivewhl_l_joint</left_joint>
-        <right_joint>drivewhl_r_joint</right_joint>
-        <!-- kinematics -->
-        <wheel_separation>0.4</wheel_separation>
-        <wheel_radius>0.2</wheel_radius>
-        <!-- limits -->
-        <max_linear_acceleration>0.1</max_linear_acceleration>
-        <!-- input -->
-        <topic>/demo/cmd_vel</topic>
-        <!-- output -->
-        <odom_topic>/demo/odom</odom_topic>
-        <tf_topic>/tf</tf_topic>
-        <frame_id>odom</frame_id>
-        <child_frame_id>base_link</child_frame_id>
-    </plugin>
-    <plugin
-        filename="gz-sim-joint-state-publisher-system"
-        name="gz::sim::systems::JointStatePublisher">
-        <topic>joint_states</topic>
-    </plugin>
+    </gazebo>
 </robot>

File: isaac_ros-dev/src/sim/description/custom_robot/robot.urdf.xacro (robot description, xacro)
@@ -4,3 +4,6 @@
     <xacro:include filename="gazebo_control.xacro"/>
     <xacro:include filename="camera.xacro"/>
+    <xacro:include filename="imu.xacro"/>
+    <xacro:include filename="depth_camera.xacro"/>
+    <xacro:include filename="lidar.xacro"/>
 </robot>
