Commit message: the sim hates me I hate the sim in a way we see eye to eye

File: isaac_ros-dev/src/sim/description/custom_robot/camera.xacro (robot description, xacro)
@@ -4,5 +4,5 @@
         <parent link="chassis"/>
         <child link="camera_link"/>
-        <origin xyz="0.4191 0 0.275" rpy="0 0 0"/>
+        <origin xyz="0.4191 0 0.275" rpy="0 -0.785 0"/>
     </joint>
     <link name="camera_link">
@@ -22,5 +22,5 @@
         <parent link="camera_link"/>
         <child link="camera_link_optical"/>
-        <origin xyz="0 0 0" rpy="${-pi/2} ${-pi/4} ${-pi/2}"/>
+        <origin xyz="0 0 0" rpy="${-pi/2} 0 ${-pi/2}"/>
     </joint>
     <link name="camera_link_optical"></link>
@@ -28,5 +28,5 @@
         <material>Gazebo/Red</material>
         <sensor name="camera" type="camera">
-            <pose> 0 0 0 0 -1.5 0 </pose>
+            <pose> 0 0 0 0 0 0 </pose>
             <visualize>true</visualize>
             <update_rate>10</update_rate>

File: isaac_ros-dev/src/sim/description/custom_robot/depth_camera.xacro (robot description, xacro)
@@ -23,5 +23,5 @@
     <parent link="base_link"/>
     <child link="depth_camera_link"/>
-    <origin xyz="0.215 0 0.05" rpy="0 0 0"/>
+    <origin xyz="0.415 0 0.35" rpy="0 0 0"/>
     </joint>
     <link name="camera_depth_frame"/>

File: isaac_ros-dev/src/sim/description/custom_robot/gazebo_control.xacro (robot description, xacro)
@@ -15,5 +15,5 @@
             <robot_base_frame>base_link</robot_base_frame>
             <publish_odom>true</publish_odom>
-            <publish_odom_tf>true</publish_odom_tf>
+            <publish_odom_tf>false</publish_odom_tf>
             <publish_wheel_tf>true</publish_wheel_tf>
         </plugin>

File: isaac_ros-dev/src/sim/description/custom_robot/imu.xacro (robot description, xacro)
@@ -26,6 +26,5 @@
             <plugin filename="libgazebo_ros_imu_sensor.so" name="imu_plugin">
                 <ros>
-                    <namespace>/autonav</namespace>
-                    <remapping>~/out:=/imu</remapping>
+                    <remapping>~/out:=imu</remapping>
                 </ros>
                 <initial_orientation_as_reference>false</initial_orientation_as_reference>
@@ -34,6 +33,4 @@
             <update_rate>100</update_rate>
             <visualize>true</visualize>
-            <topic>demo/imu</topic>
-            <gz_frame_id>imu_link</gz_frame_id>
             <imu>
                 <angular_velocity>

File: isaac_ros-dev/src/sim/description/custom_robot/lidar.xacro (robot description, xacro)
@@ -3,5 +3,5 @@
     <link name="lidar_link">
     <inertial>
-        <origin xyz="0 0 0" rpy="0 0 0"/>
+        <origin xyz="0 0 1" rpy="0 0 0"/>
         <mass value="0.125"/>
         <inertia ixx="0.001"  ixy="0"  ixz="0" iyy="0.001" iyz="0" izz="0.001" />

Commit message: two sounds... me slam you and you slam the floor

File: isaac_ros-dev/src/sim/description/custom_robot/camera.xacro (robot description, xacro)
@@ -4,5 +4,5 @@
         <parent link="chassis"/>
         <child link="camera_link"/>
-        <origin xyz="0.4191 0 0.275" rpy="0 -0.785 0"/>
+        <origin xyz="0.4191 0 0.275" rpy="0 0.485 0"/>
     </joint>
     <link name="camera_link">

File: isaac_ros-dev/src/sim/description/custom_robot/gazebo_control.xacro (robot description, xacro)
@@ -3,4 +3,7 @@
     <gazebo>
         <plugin name="diff_drive" filename="libgazebo_ros_diff_drive.so">
+            <ros>
+                <namespace>/</namespace>
+            </ros>
             <!--WHEEL INFORMATION-->
             <left_joint>left_wheel_joint</left_joint>

File: isaac_ros-dev/src/sim/description/custom_robot/robot_core.xacro (robot description, xacro)
@@ -1,5 +1,13 @@
 <?xml version="1.0"?>
 <robot xmlns:xacro="http://www.ros.org/wiki/xacro" >
+    <xacro:property name="base_width" value="0.31"/>
+    <xacro:property name="base_length" value="0.42"/>
+    <xacro:property name="base_height" value="0.18"/>
     <xacro:include filename="inertial_macros.xacro"/>
+    <xacro:property name="wheel_radius" value="0.10"/>
+    <xacro:property name="wheel_width" value="0.04"/>
+    <xacro:property name="wheel_ygap" value="0.025"/>
+    <xacro:property name="wheel_zoff" value="0.05"/>
+    <xacro:property name="wheel_xoff" value="0.12"/>
     <material name="white">
         <color rgba="1 1 1 1"/>
@@ -21,4 +29,11 @@
     </link>
     <!--END OF BASE LINK-->
+    <!-- Robot Footprint -->
+    <link name="base_footprint"/>
+    <joint name="base_joint" type="fixed">
+        <parent link="base_link"/>
+        <child link="base_footprint"/>
+        <origin xyz="0.0 0.0 ${-(wheel_radius+wheel_zoff)}" rpy="0 0 0"/>
+    </joint>
     <!--START OF CHASSIS LINK-->
     <joint name="chassis_joint" type="fixed">
@@ -49,9 +64,4 @@
             <origin xyz="0 0 0" rpy="0 0 0"/>
         </xacro:inertial_box>
-        <inertial>
-            <mass value="5.0"/>
-            <origin xyz="0 0 0" rpy="0 0 0"/>
-            <inertia ixx="0.1" ixy="0.0" ixz="0.0" iyy="0.1" iyz="0.0" izz="0.1"/>
-        </inertial>
     </link>
     <gazebo reference="chassis">
