Commit message: lets freaking go

File: isaac_ros-dev/src/bringup/description/bowser.urdf.xacro (robot description, xacro)
@@ -16,9 +16,9 @@
     <origin xyz="0.4 0.0 0.3" rpy="0 0.785398 0"/>
   </joint>
-  <link name="lidar_footprint"/>
+  <link name="lidar_footprint_6"/>
   <joint name="lidar_joint" type="fixed">
     <parent link="base_link"/>
-    <child link="lidar_footprint"/>
-    <origin xyz="0.44 0.0 0.15" rpy="0 3.14159 0"/>
+    <child link="lidar_footprint_6"/>
+    <origin xyz="0.44 0.0 0.15" rpy="3.1415 0 0"/>
   </joint>
   <link name="gps_footprint"/>

Commit message: who forgot to commit all this code

File: isaac_ros-dev/src/bringup/description/bowser.urdf.xacro (robot description, xacro)
@@ -10,14 +10,14 @@
     <origin xyz="0.0 0.0 0.0" rpy="0 0 0"/>
   </joint>
-  <link name="camera_footprint"/>
-  <joint name="camera_joint" type="fixed">
+  <link name="zed_camera_link"/>
+  <joint name="zed_camera_joint" type="fixed">
     <parent link="base_link"/>
-    <child link="camera_footprint"/>
+    <child link="zed_camera_link"/>
     <origin xyz="0.4 0.0 0.3" rpy="0 0.785398 0"/>
   </joint>
-  <link name="lidar_footprint_6"/>
+  <link name="lidar_footprint"/>
   <joint name="lidar_joint" type="fixed">
     <parent link="base_link"/>
-    <child link="lidar_footprint_6"/>
+    <child link="lidar_footprint"/>
     <origin xyz="0.44 0.0 0.15" rpy="3.1415 0 0"/>
   </joint>
